Commit message: fix stl coor

File: urdf/lamp.urdf (robot description, URDF)
Before this commit: robot lamp, 5 links, 4 joints
Links:
- link base: geometry visual mesh filename=package://pixar/meshes/base.stl scale=0.01 0.01 0.01
- link head: geometry visual mesh filename=package://pixar/meshes/head.stl scale=0.01 0.01 0.01
- link link0: geometry visual mesh filename=package://pixar/meshes/link.stl scale=0.01 0.01 0.01
- link link1: geometry visual mesh filename=package://pixar/meshes/link.stl scale=0.01 0.01 0.01
- link link2: geometry visual mesh filename=package://pixar/meshes/link.stl scale=0.01 0.01 0.01
Joints:
- joint theta2: origin xyz=0 0 0 rpy=0 0 0 -> xyz=0 0 0.5 rpy=0 0 0
- joint theta3: origin xyz=0 0 0 rpy=0 0 0 -> xyz=0 0 0.5 rpy=0 0 0
- joint theta4: origin xyz=0 0 0 rpy=0 0 0 -> xyz=0 0 0.5 rpy=0 0 0

Commit message: add scene, code cleanup

File: urdf/lamp.urdf (robot description, URDF)
Before this commit: robot lamp, 5 links, 4 joints
Links:
- link base: geometry visual mesh filename=package://pixar/meshes/lamp/base.stl scale=0.01 0.01 0.01
- link head: geometry visual mesh filename=package://pixar/meshes/lamp/head.stl scale=0.01 0.01 0.01
- link link0: geometry visual mesh filename=package://pixar/meshes/lamp/link.stl scale=0.01 0.01 0.01
- link link1: geometry visual mesh filename=package://pixar/meshes/lamp/link.stl scale=0.01 0.01 0.01
- link link2: geometry visual mesh filename=package://pixar/meshes/lamp/link.stl scale=0.01 0.01 0.01

Commit message: fix path issues

File: urdf/lamp.urdf (robot description, URDF)
Before this commit: robot lamp, 5 links, 4 joints
Links:
- link base: geometry visual mesh filename=package://pixar/meshes/base.stl scale=0.01 0.01 0.01
- link head: geometry visual mesh filename=package://pixar/meshes/head.stl scale=0.01 0.01 0.01
- link link0: geometry visual mesh filename=package://pixar/meshes/link.stl scale=0.01 0.01 0.01
- link link1: geometry visual mesh filename=package://pixar/meshes/link.stl scale=0.01 0.01 0.01
- link link2: geometry visual mesh filename=package://pixar/meshes/link.stl scale=0.01 0.01 0.01

Commit message: fix everything

File: urdf/lamp.urdf (robot description, URDF)
Before this commit: robot lamp, 5 links, 4 joints
Links:
- link base: geometry visual mesh filename=package://pixar/meshes/base.dae scale=0.01 0.01 0.01
- link head: geometry visual mesh filename=package://pixar/meshes/headog.dae scale=10 10 10
- link link0: geometry visual mesh filename=package://pixar/meshes/linkog.dae scale=10 10 10
- link link1: geometry visual mesh filename=package://pixar/meshes/linkog.dae scale=10 10 10
- link link2: geometry visual mesh filename=package://pixar/meshes/linkog.dae scale=10 10 10
Joints:
- joint theta1: origin xyz=0 0 0 rpy=0 0 0 -> xyz=0 0 0.1 rpy=0 0 0

Commit message: change name

File: urdf/lamp.urdf (robot description, URDF)
Before this commit: robot lamp, 5 links, 4 joints
Links:
- link head: geometry visual mesh filename=package://pixar/meshes/head.dae scale=10 10 10
- link link0: geometry visual mesh filename=package://pixar/meshes/link.dae scale=10 10 10
- link link1: geometry visual mesh filename=package://pixar/meshes/link.dae scale=10 10 10
- link link2: geometry visual mesh filename=package://pixar/meshes/link.dae scale=10 10 10

Commit message: fix namespace issue

File: urdf/lamp.urdf (robot description, URDF)
Before this commit: robot lamp, 5 links, 4 joints
Links:
- added link head_theta4; visual box size=0 0 0
Joints:
- added joint theta5: type continuous, parent head_theta4, child head, origin xyz=0 0 0 rpy=0 0 0, axis 1 0 0
- joint theta4: child head -> head_theta4

Commit message: Fixed Jacobian. Added COM plotting. It jumps

File: urdf/lamp.urdf (robot description, URDF)
Before this commit: robot lamp, 6 links, 5 joints
Joints:
- joint theta1: origin xyz=0 0 0.1 rpy=0 0 0 -> xyz=0 0 0 rpy=0 0 0
